File: HARDWARE/HARDWARE.sch (KiCad schematic (older format))
At the start: 2 parts

Commit message: 13/07/2021
Parts:
- added C1, C2: 2u2F, Capacitor_THT:CP_Radial_Tantal_D4.5mm_P2.50mm, symbol Device:CP_Small
- added C10, C11, C12: 100nF, Capacitor_SMD:C_0805_2012Metric, symbol Device:C_Small
- added C13, C15: 100nF, Capacitor_SMD:C_0805_2012Metric, symbol Device:C
- added C14, C9: 10uF, Capacitor_THT:CP_Radial_Tantal_D4.5mm_P2.50mm, symbol Device:CP
- added C3, C4, C5, C6, C7, C8: 10uF, Capacitor_THT:CP_Radial_Tantal_D4.5mm_P2.50mm, symbol Device:CP_Small
- added D1: LED, Resistor_SMD:R_0603_1608Metric, symbol Device:LED
- added J1: RedPitaya, Connector_IDC:IDC-Header_2x13_P2.54mm_Vertical, symbol Connector_Generic:Conn_02x13_Counter_Clockwise
- added J2: GPS, Connector_PinSocket_2.54mm:PinSocket_1x06_P2.54mm_Vertical, symbol Connector_Generic:Conn_01x06
- added J3: RJ45_PMT, Connector_RJ:RJ45_Amphenol_54602-x08_Horizontal, symbol Connector:RJ45
- added J4: TEST_POINT, Connector_PinHeader_2.54mm:PinHeader_1x05_P2.54mm_Vertical, symbol Connector_Generic:Conn_01x05
- added J5: RJ11_BMP180, Connector_RJ:RJ14_Connfly_DS1133-S4_Horizontal, symbol Connector:4P4C
- added R1: 5.1k, Resistor_SMD:R_0603_1608Metric, symbol Device:R
- added R2: 3k, Resistor_SMD:R_0603_1608Metric, symbol Device:R
- added R3: 330, Resistor_SMD:R_0603_1608Metric, symbol Device:R
- added R4: 100k, Resistor_SMD:R_0603_1608Metric, symbol Device:R
- added U1: MAX662ACSA+, Max662A:MAX662ACSA&plus_, symbol MAX662A:MAX662ACSA+
- added U2: TLV5616CD, TLV5616CD:SOIC127P599X175-8N, symbol TLV5616CD:TLV5616CD
- added U5: LM358, Package_SO:SOIC-8_3.9x4.9mm_P1.27mm, symbol Amplifier_Operational:LM358
- U3, U4: renamed from U?; footprint (none) -> Package_DIP:DIP-8_W7.62mm
Connections:
- net 5V_UNREG: now reaches U3.1 (IN)
- net 5V_UNREG: now also U3.4 (~OFF), C3.1, J1.26 (Pin_26)
- net GND: now reaches U3.2 (GND), U3.3 (GND), U3.6 (GND), U3.7 (GND)
- net GND: now also U3.5 (SET), U4.2 (GND), U4.3 (GND), U4.5 (SET), U4.6 (GND), U4.7 (GND), C10.2, C11.2, C12.2, C13.2, C14.2, C15.2, C3.2, C4.2, C5.2, C6.2, C7.2, C8.2, C9.2, J1.1 (Pin_1), J1.15 (Pin_15), J1.16 (Pin_16), J1.2 (Pin_2), J1.5 (Pin_5), J1.6 (Pin_6), J2.5 (Pin_5), J3.4, J4.5 (Pin_5), J5.2, R2.2, R3.2, U1.7 (GND), U1.8 (SHDN), U2.3 (~CS), U2.5 (AGND), U5.4 (V-)
- net +5V: now reaches U3.8 (OUT)
- net +5V: now also U4.1 (IN), U4.4 (~OFF), C10.1, C4.1, C5.1, C6.1, J2.6 (Pin_6), J3.5, J4.3 (Pin_3), U1.5 (VCC)
- net +3V3: now reaches U4.8 (OUT)
- net +3V3: now also C11.1, C13.1, C7.1, C9.1, D1.2 (A), J4.2 (Pin_2), J5.1, R1.1, U2.8 (VDD), U5.8 (V+)
- new net: C1.2, U1.1 (C1-)
- new net: C1.1, U1.2 (C1+)
- new net: C2.2, U1.3 (C2-)
- new net: C2.1, U1.4 (C2+)
- new net: R1.2, R2.1, U2.6 (REFIN)
- new net: R4.2, U5.1, U5.2 (-)
- new net: C14.1, R4.1, U5.5 (+)
- new net: D1.1 (K), R3.1
- new net +12V: C12.1, C8.1, J3.6, J4.4 (Pin_4), U1.6 (VOUT)
- new net GPS_RXD: J1.19 (Pin_19), J2.3 (Pin_3)
- new net GPS_TXD: J1.20 (Pin_20), J2.4 (Pin_4)
- new net I2C_SCL: J1.18 (Pin_18), J5.3
- new net I2C_SDA: J1.17 (Pin_17), J5.4
- new net OUT_REF: U2.7 (OUT), U5.3 (+)
- new net PMT_CTRL_V: C15.1, J3.3, J4.1 (Pin_1), U5.6 (-), U5.7
- new net PPS: J2.1 (Pin_1), J2.2 (Pin_2)
- new net SPI_CLK: J1.22 (Pin_22), U2.2 (SCLK)
- new net SPI_CS: J1.21 (Pin_21), U2.4 (FS)
- new net SPI_MOSI: J1.24 (Pin_24), U2.1 (DIN)
- no-connect marks 0 -> 14
Other:
- note added: "2.7 V - 5.5 V low power 12 Bit DAC"
- note added: "Connector for GPS module"
- note added: "Connector for PMT circuit board"
- note added: "DC-DC converter charge-up: 5 VDC - 12 V DC"
- note added: "LDO, Linear Voltage Regulator: 5 V DC - 3.3 V DC"
- note added: "LDO, Linear Voltage Regulator: 5 V DC - 5 V DC"
- note added: "LED power on indicator"
- note added: "RJ11 connector for: \nBMP180 sensor"
- note added: "Red Pitaya Connector"
- note added: "Test Point for: PMT Voltage, \n3.3 V, 5 V, 12 V and GND"
- note added: "Variable voltage signal adjustment with low pass filter"
- moved on the sheet: U3, U4
