File: HARDWARE/HARDWARE.kicad_pcb (KiCad board)
At the start: 2 copper layers, 55.9 x 57.1 mm, 31 parts, among them J1 RedPitaya, J2 GPS, J3 RJ45_PMT, J4 TEST_POINT, J5 RJ11_BMP180, U1 MAX662ACSA+, U2 TLV5616CD, U3 MAX603, U4 MAX604, U5 LM358

Commit message: 14/07/2021
Parts:
- turned R3 to 0 degrees
Routing:
- net GND: track 41.6 -> 240.9 mm
- net /GPS_RXD: track 56.9 -> 55.0 mm
- net Net-(D1-Pad1): track 3.22 -> 2.54 mm
- net (no net): vias 3 -> 4
